File: GL-0811A.kicad_pcb (KiCad board)
At the start: 2 copper layers, 38.1 x 76.2 mm, 1 part

Commit message: 28.03/2
Parts:
- removed REF**: R+SW, GL-0811A:R+SW
- added C1: C, GL-0811A:C1, F.Cu at (53.6, 92.7)
- added C2: C, GL-0811A:C1, F.Cu at (66.0, 77.0)
- added C3: C, GL-0811A:C1, F.Cu at (76.1, 109.7)
- added C4: C, GL-0811A:C1, F.Cu at (59.7, 92.7)
- added FU1: F1, GL-0811A:Fuse, F.Cu at (56.0, 141.0)
- added FU2: F1, GL-0811A:Fuse2, F.Cu at (59.7, 123.0)
- added FU3: F1, GL-0811A:Fuse2, F.Cu at (75.1, 97.6)
- added R1: R+SW, GL-0811A:R+SW, F.Cu at (64.0, 109.3)
- added R2: R, GL-0811A:R_Axial_DIN0207_L6.3mm_D2.5mm_P10.16mm_Horizontal, F.Cu at (65.5, 130.9)
- added R3: R, GL-0811A:R_Axial_DIN0207_L6.3mm_D2.5mm_P10.16mm_Horizontal, F.Cu at (69.6, 130.9)
- added R4: R+SW, GL-0811A:R+SW, F.Cu at (72.0, 142.0)
- added R5: R, GL-0811A:R_Axial_DIN0207_L6.3mm_D2.5mm_P10.16mm_Horizontal, F.Cu at (72.5, 80.6)
- added R6: R, GL-0811A:R_Axial_DIN0207_L6.3mm_D2.5mm_P10.16mm_Horizontal, F.Cu at (77.0, 81.0)
- added U2: Semistor, GL-0811A:sem1, F.Cu at (55.6, 123.4)
- added U4: Semistor, GL-0811A:sem2, F.Cu at (76.0, 88.0)
- added X4: CONN_3, GL-0811A:CON1, F.Cu at (77.6, 125.3)
Other:
- board size 38.1 x 76.2 mm -> 30 x 90 mm
